File: Devboard-G070-32pins.kicad_pcb (KiCad board)
At the start: 2 copper layers, 10 parts, among them Q3 2N7002H, U1 STM32G070KBTx, U2 TLV70233_SOT23-5

Commit message: schematic update
Parts:
- moved U1 22.6 mm to (131.3, 76.5)
- moved Q3 19.0 mm to (116.6, 69.0)
Routing:
- net GND: track 0.00 -> 14.4 mm
Changed lines of the file:
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@@
 	(footprint "Package_TO_SOT_SMD:SOT-23"
 		(layer "F.Cu")
-		(at 98.675 75.395)
+		(at 116.5625 69)
 		(descr "SOT, 3 Pin (https://www.jedec.org/system/files/docs/to-236h.pdf variant AB), generated with kicad-footprint-generator ipc_gullwing_generator.py")
 		(tags "SOT TO_SOT_SMD")
@@
 	(footprint "Package_QFP:LQFP-32_7x7mm_P0.8mm"
 		(layer "F.Cu")
-		(at 108.825 78.7)
+		(at 131.325 76.5)
 		(descr "LQFP, 32 Pin (https://www.nxp.com/docs/en/package-information/SOT358-1.pdf), generated with kicad-footprint-generator ipc_gullwing_generator.py")
 		(tags "LQFP QFP")
@@
 		)
 	)
+	(segment
+		(start 115.625 69.95)
+		(end 122.575 76.9)
+		(width 0.2)
+		(layer "F.Cu")
+		(net 17)
+	)
+	(segment
+		(start 122.575 76.9)
+		(end 127.15 76.9)
+		(width 0.2)
+		(layer "F.Cu")
+		(net 17)
+	)
 )
