File: Devboard-G070-32pins.kicad_pcb (KiCad board)
At the start: 2 copper layers, 17 parts, among them J1 Conn_01x05, J2 Conn_01x07, J4 Conn_01x07, J5 Conn_01x02, SW1 SW_MEC_5E, SW3 SW_MEC_5E, U2 STM32G070KBTx

Commit message: [feat] PCB routing
Parts:
- C1: value C -> 100nF; footprint Capacitor_THT:C_Radial_D6.3mm_H5.0mm_P2.50mm -> Capacitor_THT:C_Disc_D3.0mm_W1.6mm_P2.50mm
- C2: value C -> 100nF; footprint Capacitor_SMD:C_0402_1005Metric_Pad0.74x0.62mm_HandSolder -> Capacitor_THT:C_Disc_D3.0mm_W1.6mm_P2.50mm
- D1: footprint LED_THT:LED_D1.8mm_W1.8mm_H2.4mm_Horizontal_O3.81mm_Z4.9mm -> LED_THT:LED_D2.0mm_W4.8mm_H2.5mm_FlatTop
- R2: value R -> 1k
- SW1, SW3: footprint Button_Switch_SMD:SW_MEC_5GSH9 -> Button_Switch_THT:SW_PUSH-12mm_Wuerth-430476085716
- moved D2 85.8 mm to (135.0, 163.3), turned to 90 degrees
- moved R3 75.0 mm to (126.3, 163.6), turned to 180 degrees
- moved J4 72.9 mm to (118.2, 135.5), turned to -90 degrees
- moved R4 68.0 mm to (126.3, 159.6), turned to 180 degrees
- moved J2 66.6 mm to (118.2, 171.0), turned to -90 degrees
- moved SW3 61.7 mm to (86.8, 163.5), turned to 180 degrees
- moved R5 61.1 mm to (126.3, 155.5), turned to 180 degrees
- moved R1 51.5 mm to (92.2, 164.8), turned to 90 degrees
- moved SW1 46.3 mm to (74.2, 143.0), turned to 0 degrees
- moved C2 41.7 mm to (96.8, 162.2), turned to 90 degrees
- moved C1 30.8 mm to (91.0, 147.8), turned to -90 degrees
- moved J1 23.3 mm to (69.0, 164.6), turned to 180 degrees
- moved BZ1 17.9 mm to (126.0, 149.3), turned to 90 degrees
- moved U2 17.8 mm to (104.0, 152.0), turned to 0 degrees
- moved R2 15.3 mm to (87.3, 135.5), turned to 180 degrees
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Connections:
- C1 pad 1: NRST -> GND
- C1 pad 2: GND -> NRST
- J1 pad 1: +3V3 -> SWDIO
- J1 pad 2: NRST -> SWCLK
- J1 pad 3: SWCLK -> NRST
- J1 pad 4: SWDIO -> +3V3
- J2 pad 10: PA0 -> PA2
- J2 pad 11: PC15 -> PA1
- J2 pad 2: PB1 -> PA10
- J2 pad 3: PB0 -> PB1
- J2 pad 4: PA6 -> PB0
- J2 pad 5: PA5 -> PA7
- J2 pad 6: PA4 -> PA6
- J2 pad 7: PA2 -> PA5
- J2 pad 8: PA3 -> PA4
- J2 pad 9: PA1 -> PA3
- J4 pad 1: PA10 -> PA9
- J4 pad 10: PB9 -> PC14
- J4 pad 11: PC14 -> PC15
- J4 pad 3: PA9 -> PB3
- J4 pad 4: PB3 -> PB4
- J4 pad 5: PB4 -> PB5
- J4 pad 6: PB5 -> PB6
- J4 pad 7: PB6 -> PB7
- J4 pad 8: PB7 -> PB8
- J4 pad 9: PB8 -> PB9
- J5 pad 1: +3V5 -> +3V3
- SW1 pad 1: GND -> NRST
- SW1 pad 2: GND -> NRST
- U2 pad 14: Buzzer -> PA7
- U2 pad 17: LED_B -> LED_R
- U2 pad 18: LED_R -> LED_G
- U2 pad 19: LED_G -> LED_B
- U2 pad 21: PA10 -> Buzzer
- U2 pad 23: BTN_Code -> PA10
- U2 pad 7: PA0 -> BTN_Code
Routing:
- net GND: track 0.21 -> 268.1 mm, vias 0 -> 4
- net +3V3: track 0.00 -> 64.3 mm, vias 0 -> 1
- net SWDIO: track 0.00 -> 57.0 mm, vias 0 -> 1
- net SWCLK: track 0.00 -> 51.5 mm, vias 0 -> 1
- net NRST: track 0.00 -> 43.7 mm
- net PC6: track 0.03 -> 32.9 mm, vias 0 -> 1
- net PA10: track 0.00 -> 28.2 mm, vias 0 -> 1
- net PA9: track 0.00 -> 24.3 mm
- net PC15: track 0.00 -> 20.0 mm
- net PA1: track 0.00 -> 19.6 mm
- net Buzzer: track 0.42 -> 19.5 mm
- net PC14: track 0.00 -> 18.0 mm
- net PB1: track 0.00 -> 17.4 mm
- net PA2: track 0.00 -> 17.3 mm
- net PB0: track 0.00 -> 16.7 mm
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
Commit message: Modifying footprint positions
Parts:
- SW1, SW3: footprint Button_Switch_THT:SW_PUSH-12mm_Wuerth-430476085716 -> personalized:SW_PUSH-12mm
- moved J1 69.4 mm to (132.0, 135.5), turned to 0 degrees
- moved R2 16.2 mm to (93.0, 150.7), turned to 90 degrees
- moved D2 15.2 mm to (121.1, 169.5), turned to 0 degrees
- moved D1 11.9 mm to (86.2, 135.5)
- moved J5 11.5 mm to (71.0, 135.5), turned to 0 degrees
- moved SW3 10.4 mm to (80.5, 155.2)
- moved R5 9.55 mm to (127.2, 165.0), turned to 90 degrees
- moved R1 8.84 mm to (93.0, 156.0), turned to -90 degrees
- moved C2 7.63 mm to (90.1, 158.5)
- moved SW1 6.33 mm to (80.5, 142.0), turned to 180 degrees
- moved R4 5.84 mm to (124.2, 165.0), turned to 90 degrees
- moved BZ1 5.66 mm to (123.0, 144.5), turned to -90 degrees
- moved R3 5.30 mm to (121.2, 165.0), turned to 90 degrees
- moved C1 3.08 mm to (90.1, 150.7)
Connections:
- net PA9 renamed PA11
- C2 pad 1: Net-(C2-Pad1) -> GND
- J1 pad 1: SWDIO -> +3V3
- J1 pad 3: NRST -> SWDIO
- J1 pad 4: +3V3 -> NRST
- J2 pad 1: PC6 -> PA8
- J2 pad 2: PA10 -> PB2
- R1 pad 2: Net-(C2-Pad1) -> GND
- U2 pad 17: LED_R -> PB2
- U2 pad 18: LED_G -> PA8
- U2 pad 19: LED_B -> LED_R
- U2 pad 20: PC6 -> LED_G
- U2 pad 21: Buzzer -> LED_B
- U2 pad 23: PA10 -> Buzzer
Routing:
- net GND: track 268.1 -> 387.5 mm
- net PA11: track 24.3 -> 64.2 mm
- net +3V3: track 64.3 -> 100.4 mm, vias 1 -> 0
- net PC6: track 32.9 -> 0.00 mm, vias 1 -> 0
- net SWDIO: track 57.0 -> 27.4 mm, vias 1 -> 0
- net PA10: track 28.2 -> 0.00 mm, vias 1 -> 0
- net NRST: track 43.7 -> 71.8 mm
- net PA8: track 0.00 -> 22.8 mm
- net SWCLK: track 51.5 -> 29.3 mm, vias 1 -> 0
- net PB2: track 0.00 -> 20.8 mm
- net BTN_Code: track 8.39 -> 28.3 mm
- net Net-(R1-Pad1): track 6.04 -> 24.9 mm
- net LED_B: track 11.5 -> 21.5 mm
- net Net-(C2-Pad1): track 8.68 -> 0.00 mm
- net Net-(D1-A): track 2.80 -> 9.33 mm
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
Commit message: done - V1
Parts:
- added C3: 100uF, Capacitor_THT:CP_Radial_D8.0mm_P3.50mm, F.Cu at (21.3, 14.7)
- added C4: 22pF, Capacitor_THT:CP_Radial_Tantal_D4.5mm_P5.00mm, F.Cu at (27.5, 16.5)
- added H1: fixing hole, MountingHole:MountingHole_3mm_Pad, F.Cu at (0.00, 21.6)
- added H2: fixing hole, MountingHole:MountingHole_3mm_Pad, F.Cu at (80.0, 21.6)
- added J3: Conn_01x01, TestPoint:TestPoint_THTPad_1.0x1.0mm_Drill0.5mm, F.Cu at (53.3, 18.8)
- added J6: NS6312, Connector_PinHeader_2.54mm:PinHeader_1x03_P2.54mm_Vertical, F.Cu at (15.8, 10.5)
- added J7: Conn_01x03, Connector_PinHeader_2.54mm:PinHeader_1x03_P2.54mm_Vertical, F.Cu at (12.0, 10.5)
- added Q1: 2N7002H, Package_TO_SOT_THT:TO-251-3_Vertical, F.Cu at (73.6, 22.2)
- added R6: 100, Resistor_THT:R_Axial_DIN0207_L6.3mm_D2.5mm_P7.62mm_Horizontal, F.Cu at (69.8, 26.2)
- added R7: 100, Resistor_THT:R_Axial_DIN0207_L6.3mm_D2.5mm_P7.62mm_Horizontal, F.Cu at (73.3, 26.2)
- J5: value Conn_01x02 -> HW-769; footprint Connector_PinHeader_2.54mm:PinHeader_1x02_P2.54mm_Vertical -> Connector_PinHeader_2.54mm:PinHeader_1x05_P2.54mm_Vertical
- moved R2 153.2 mm to (27.2, 12.3)
- moved D1 146.0 mm to (21.2, 4.80)
- moved BZ1 145.7 mm to (61.3, 12.5)
- moved R3 145.0 mm to (59.4, 33.8)
- moved D2 145.0 mm to (59.4, 38.3)
- moved J2 145.0 mm to (56.5, 39.8)
- moved U2 145.0 mm to (42.3, 20.8)
- moved R4 144.9 mm to (62.7, 33.8)
- moved R5 144.8 mm to (65.9, 33.8)
- moved J5 144.5 mm to (8.00, 5.43)
- moved J4 144.5 mm to (56.5, 4.84)
- moved J1 144.4 mm to (70.3, 4.97)
- moved C1 141.4 mm to (23.8, 25.8)
- moved C2 141.4 mm to (23.8, 33.6)
- moved SW1 141.1 mm to (13.8, 17.6)
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Connections:
- BZ1 pad 1: Buzzer -> +3V3
- BZ1 pad 2: GND -> Net-(BZ1--)
- J4 pad 1: PA11 -> PA12
- J5 pad 1: +3V3 -> VBUS
- J5 pad 2: GND -> D-
- U2 pad 22: PA11 -> Buzzer
- U2 pad 23: Buzzer -> PA12
Routing:
- net PA11: track 64.2 -> 0.00 mm
- net GND: track 387.5 -> 357.9 mm
- net PA12: track 0.00 -> 23.4 mm
- net Buzzer: track 17.1 -> 35.5 mm
- net +3V3: track 100.4 -> 117.2 mm
- net NRST: track 71.8 -> 87.1 mm
- net VBUS: track 0.00 -> 10.1 mm
- net Net-(BZ1--): track 0.00 -> 8.57 mm
- net BTN_Code: track 28.3 -> 36.3 mm
- net Net-(Q1-G): track 0.00 -> 7.62 mm
- net Net-(D1-A): track 9.33 -> 3.53 mm
- net D-: track 0.00 -> 5.05 mm
- net D+: track 0.00 -> 5.05 mm
- net DI: track 0.00 -> 5.05 mm
- net Net-(R1-Pad1): track 24.9 -> 27.1 mm
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Other:
- board outline added: 88.3 x 44 mm

Commit message: bugs
Parts:
- added R8: 4.7k, Resistor_THT:R_Axial_DIN0207_L6.3mm_D2.5mm_P7.62mm_Horizontal, F.Cu at (31.5, 27.2)
- D2: footprint LED_THT:LED_D5.0mm-4_RGB_Wide_Pins -> personalized:LED_RGB
- moved R6 7.62 mm to (70.0, 33.8), turned to 90 degrees
- moved C3 7.07 mm to (28.0, 12.5)
- moved R2 6.87 mm to (21.2, 15.6)
- moved D2 4.08 mm to (63.5, 38.5)
- moved D1 2.56 mm to (23.8, 5.00), turned to 180 degrees
- moved J5 1.15 mm to (7.50, 4.39)
- moved J6 1.15 mm to (15.3, 9.47)
- moved J7 1.15 mm to (11.5, 9.47)
- moved R4 0.84 mm to (63.5, 33.8)
- moved R3 0.84 mm to (60.3, 33.8)
- moved R5 0.84 mm to (66.8, 33.8)
- moved C4 0.50 mm to (28.0, 16.5)
- moved SW1 0.39 mm to (13.8, 18.0)
- moved Q1 0.30 mm to (73.3, 22.2)
Routing:
- net +3V3: track 117.2 -> 219.3 mm
- net Buzzer: track 35.5 -> 26.3 mm
- net Net-(Q1-G): track 7.62 -> 13.0 mm
- net Net-(R1-Pad1): track 27.1 -> 24.6 mm
- net GND: track 357.9 -> 355.5 mm, vias 4 -> 0
- net LED_G: track 18.1 -> 20.0 mm
- net LED_B: track 21.5 -> 23.2 mm
- net LED_R: track 14.8 -> 16.4 mm
- net PB9: track 15.8 -> 14.6 mm
- net PC15: track 19.4 -> 18.6 mm
- net NRST: track 87.1 -> 87.8 mm
- net PC14: track 17.2 -> 16.6 mm
- net PA8: track 22.8 -> 22.2 mm
- net PA1: track 19.6 -> 20.1 mm
- net Net-(D1-A): track 3.53 -> 3.00 mm
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
Commit message: perf: 45° micro
Parts:
- C1, C2: footprint Capacitor_THT:C_Disc_D3.0mm_W1.6mm_P2.50mm -> personalized:C_Disc_D1mm
- C3: footprint Capacitor_THT:CP_Radial_D8.0mm_P3.50mm -> personalized:CP_Radial_1mm
- C4: footprint Capacitor_THT:CP_Radial_Tantal_D4.5mm_P5.00mm -> personalized:CP_Radial_Tantal_1mm
- D1: footprint LED_THT:LED_D2.0mm_W4.8mm_H2.5mm_FlatTop -> personalized:LED_1mm
- H1, H2: footprint MountingHole:MountingHole_3mm_Pad -> personalized:V_1mm
- J3: footprint TestPoint:TestPoint_THTPad_1.0x1.0mm_Drill0.5mm -> TestPoint:TestPoint_THTPad_D2.0mm_Drill1.0mm
- R1, R2, R3, R4, R5, R6, R7, R8: footprint Resistor_THT:R_Axial_DIN0207_L6.3mm_D2.5mm_P7.62mm_Horizontal -> personalized:Resistor_THT_Horizontal_1mm
- moved D2 85.1 mm to (-19.2, 18.3)
- moved R3 85.1 mm to (-22.4, 13.6)
- moved R4 85.1 mm to (-19.2, 13.6)
- moved R5 85.1 mm to (-16.0, 13.6)
- moved C1 60.7 mm to (-32.7, 3.66), turned to 0 degrees
- moved R6 56.9 mm to (26.4, -2.72), turned to 180 degrees
- moved J3 55.3 mm to (17.0, -22.9)
- moved C3 55.0 mm to (-25.1, -2.02), turned to -90 degrees
- moved R7 53.4 mm to (26.4, 0.67), turned to 180 degrees
- moved J2 52.3 mm to (14.2, 9.00)
- moved SW1 50.3 mm to (-36.4, 13.7), turned to -90 degrees
- moved Q1 49.0 mm to (29.2, 0.85), turned to 90 degrees
- moved C4 48.9 mm to (-16.9, -2.87)
- moved D1 48.2 mm to (-19.4, -16.4), turned to 0 degrees
- moved U2 47.1 mm to (0.00, 0.00), turned to -45 degrees
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Connections:
- J2 pad 11: PA1 -> PA9
- J4 pad 1: PA12 -> PA15
- J4 pad 10: PC14 -> PC15
- J4 pad 11: PC15 -> PA1
- J4 pad 2: PA15 -> PB3
- J4 pad 3: PB3 -> PB4
- J4 pad 4: PB4 -> PB5
- J4 pad 5: PB5 -> PB6
- J4 pad 6: PB6 -> PB7
- J4 pad 7: PB7 -> PB8
- J4 pad 8: PB8 -> PB9
- J4 pad 9: PB9 -> PC14
- U2 pad 19: LED_R -> PA9
- U2 pad 21: LED_B -> LED_R
- U2 pad 22: Buzzer -> LED_B
- U2 pad 23: PA12 -> Buzzer
Routing:
- net +3V3: track 219.3 -> 30.6 mm
- net GND: track 355.5 -> 172.4 mm
- net NRST: track 87.8 -> 49.4 mm
- net Net-(R1-Pad1): track 24.6 -> 0.00 mm
- net LED_B: track 23.2 -> 0.00 mm
- net PA12: track 22.8 -> 0.00 mm
- net PA8: track 22.2 -> 0.00 mm
- net PB2: track 20.8 -> 0.00 mm
- net PA1: track 20.1 -> 0.00 mm
- net LED_G: track 20.0 -> 0.17 mm
- net PB1: track 17.4 -> 0.00 mm
- net PA2: track 17.3 -> 0.00 mm
- net PB0: track 16.7 -> 0.00 mm
- net PA3: track 16.5 -> 0.00 mm
- net PA4: track 16.4 -> 0.00 mm
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Other:
- board size 88.3 x 44 mm -> 89.3 x 44 mm

Commit message: board v1
Parts:
- J3: footprint TestPoint:TestPoint_THTPad_D2.0mm_Drill1.0mm -> personalized:hole
- moved J3 33.6 mm to (-7.80, -0.20)
- moved R8 7.86 mm to (34.8, 2.86), turned to 90 degrees
- moved SW3 4.77 mm to (40.0, 11.9)
- moved C2 3.40 mm to (31.6, -0.56), turned to -90 degrees
- moved R1 2.75 mm to (23.6, 18.9)
- moved BZ1 2.61 mm to (25.4, -16.7)
- moved J1 2.61 mm to (34.8, -17.9)
- moved C3 2.46 mm to (-25.2, -4.48)
- moved R4 2.28 mm to (-20.0, 11.5)
- moved R5 2.28 mm to (-16.7, 11.5)
- moved R3 2.28 mm to (-23.2, 11.5)
- moved H1 2.03 mm to (-38.5, -0.50)
- moved SW1 1.76 mm to (-37.1, 12.1)
- moved D2 1.76 mm to (-19.9, 16.7)
- moved J6 1.52 mm to (-23.0, -15.4)
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Connections:
- J2 pad 1: PA8 -> PA10
- J2 pad 10: PA2 -> PA5
- J2 pad 11: PA9 -> PA4
- J2 pad 2: PB2 -> PC6
- J2 pad 3: PB1 -> PA9
- J2 pad 4: PB0 -> PA8
- J2 pad 5: PA7 -> PB2
- J2 pad 6: PA6 -> PB1
- J2 pad 7: PA5 -> PB0
- J2 pad 8: PA4 -> PA7
- J2 pad 9: PA3 -> PA6
- J3 pad 1: PA12 -> PA1
- U2 pad 10: PA3 -> LED_R
- U2 pad 20: LED_G -> PC6
- U2 pad 21: LED_R -> PA10
- U2 pad 22: LED_B -> BTN_Code
- U2 pad 7: BTN_Code -> LED_B
- U2 pad 9: PA2 -> LED_G
Routing:
- net GND: track 172.4 -> 265.9 mm
- net +3V3: track 30.6 -> 116.1 mm
- net NRST: track 49.4 -> 118.0 mm
- net BTN_Code: track 26.0 -> 52.7 mm
- net LED_R: track 0.06 -> 26.0 mm
- net Net-(R1-Pad1): track 0.00 -> 20.6 mm
- net LED_G: track 0.17 -> 20.6 mm
- net PA1: track 0.00 -> 16.4 mm
- net LED_B: track 0.00 -> 14.8 mm
- net PA10: track 0.00 -> 14.4 mm
- net PC6: track 0.00 -> 12.1 mm
- net PA4: track 0.00 -> 10.3 mm
- net PA9: track 0.00 -> 9.99 mm
- net PA5: track 0.00 -> 8.58 mm
- net PA8: track 0.00 -> 7.69 mm
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Other:
- board size 89.3 x 44 mm -> 88 x 46 mm
