File: Devboard-G070-32pins.kicad_pcb (KiCad board)
At the start: 2 copper layers, 88 x 46 mm, 28 parts, among them J1 Conn_01x05, J2 Conn_01x07, J3 Conn_01x01, J4 Conn_01x07, J5 HW-769, J6 NS6312, J7 Conn_01x03, Q1 2N7002H, SW1 SW_MEC_5E, SW3 SW_MEC_5E, U2 STM32G070KBTx

Commit message: fix: RGB LED symbol
Connections:
- D2 pad 2: Net-(D2-RK) -> Net-(D2-RA)
- D2 pad 3: Net-(D2-GK) -> Net-(D2-GA)
- D2 pad 4: Net-(D2-BK) -> Net-(D2-BA)
Changed lines of the file:
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@@
 	(net 44 "PA10")
 	(net 45 "PA1")
+	(net 46 "Net-(D2-RA)")
+	(net 47 "Net-(D2-GA)")
+	(net 48 "Net-(D2-BA)")
 	(footprint "personalized:SW_PUSH-12mm"
 		(layer "F.Cu")
@@
 			)
 		)
-		(property "Description" "RGB LED, anode/red/green/blue"
+		(property "Description" "RGB LED, cathode/red/green/blue"
 			(at 0 0 0)
 			(unlocked yes)
@@
 			(remove_unused_layers no)
 			(net 10 "GND")
-			(pinfunction "A")
+			(pinfunction "K")
 			(pintype "passive")
 		)
@@
 			(layers "*.Cu" "*.Mask")
 			(remove_unused_layers no)
-			(net 8 "Net-(D2-RK)")
-			(pinfunction "RK")
+			(net 46 "Net-(D2-RA)")
+			(pinfunction "RA")
 			(pintype "passive")
 		)
@@
 			(layers "*.Cu" "*.Mask")
 			(remove_unused_layers no)
-			(net 6 "Net-(D2-GK)")
-			(pinfunction "GK")
+			(net 47 "Net-(D2-GA)")
+			(pinfunction "GA")
 			(pintype "passive")
 		)
@@
 			(layers "*.Cu" "*.Mask")
 			(remove_unused_layers no)
-			(net 9 "Net-(D2-BK)")
-			(pinfunction "BK")
+			(net 48 "Net-(D2-BA)")
+			(pinfunction "BA")
 			(pintype "passive")
 		)
