File: ExtensionConnectors.kicad_sch (KiCad schematic)
At the start: 8 parts, among them J11 Conn_02x18, J5 Conn_01x08, J6 Conn_01x06, J7 Conn_01x10, J8 Conn_01x08, J9 Conn_02x18, U3 STM32G070KBTx

Commit message: schematic update
Parts:
- added C8: 100nf, symbol Device:C
Connections:
- net +3V3: no longer J5.2 (Pin_2)
- net GND: now also C8.2
- net at R5.2: now also J11.b4 (Pin_b4); no longer J11.b3 (Pin_b3)
- net at J9.b3 (Pin_b3): now also C8.1
- net IOREF: now reaches J11.a4 (Pin_a4)
- net IOREF: now also J5.2 (Pin_2)
Changed lines of the file:
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@@
-	)
-	(junction
-		(at 114.3 81.28)
-		(diameter 0)
-		(color 0 0 0 0)
 	)
 	(junction
@@
 	(wire
 		(pts
+			(xy 236.22 76.2) (xy 273.05 76.2)
+		)
+		(stroke
+			(width 0)
+			(type default)
+		)
+	)
+	(wire
+		(pts
 			(xy 203.2 88.9) (xy 223.52 88.9)
 		)
@@
 	(wire
 		(pts
-			(xy 104.14 81.28) (xy 114.3 81.28)
+			(xy 104.14 81.28) (xy 120.65 81.28)
 		)
 		(stroke
@@
 	(wire
 		(pts
-			(xy 91.44 73.66) (xy 87.63 73.66)
-		)
-		(stroke
-			(width 0)
-			(type default)
-		)
-	)
-	(wire
-		(pts
-			(xy 114.3 76.2) (xy 114.3 81.28)
-		)
-		(stroke
-			(width 0)
-			(type default)
-		)
-	)
-	(wire
-		(pts
-			(xy 114.3 81.28) (xy 120.65 81.28)
+			(xy 91.44 76.2) (xy 87.63 76.2)
 		)
 		(stroke
@@
 	(wire
 		(pts
+			(xy 273.05 76.2) (xy 273.05 78.74)
+		)
+		(stroke
+			(width 0)
+			(type default)
+		)
+	)
+	(wire
+		(pts
 			(xy 236.22 93.98) (xy 246.38 93.98)
 		)
@@
 	(wire
 		(pts
-			(xy 120.65 76.2) (xy 114.3 76.2)
-		)
-		(stroke
-			(width 0)
-			(type default)
-		)
-	)
-	(wire
-		(pts
 			(xy 85.09 88.9) (xy 85.09 92.71)
 		)
@@
 	(wire
 		(pts
-			(xy 87.63 53.34) (xy 87.63 73.66)
+			(xy 87.63 53.34) (xy 87.63 76.2)
 		)
 		(stroke
@@
 	(wire
 		(pts
+			(xy 104.14 76.2) (xy 120.65 76.2)
+		)
+		(stroke
+			(width 0)
+			(type default)
+		)
+	)
+	(wire
+		(pts
 			(xy 78.74 106.68) (xy 91.44 106.68)
 		)
@@
 		(pts
 			(xy 78.74 104.14) (xy 91.44 104.14)
+		)
+		(stroke
+			(width 0)
+			(type default)
+		)
+	)
+	(wire
+		(pts
+			(xy 273.05 88.9) (xy 273.05 86.36)
 		)
 		(stroke
@@
 	(label "PA3"
 		(at 87.63 111.76 180)
+		(fields_autoplaced yes)
+		(effects
+			(font
+				(size 1.27 1.27)
+			)
+			(justify right bottom)
+		)
+	)
+	(label "IOREF"
+		(at 119.38 76.2 180)
 		(fields_autoplaced yes)
 		(effects
@@
 	)
 	(symbol
+		(lib_id "Device:C")
+		(at 273.05 82.55 0)
+		(unit 1)
+		(exclude_from_sim no)
+		(in_bom yes)
+		(on_board yes)
+		(dnp no)
+		(property "Reference" "C8"
+			(at 275.336 82.55 0)
+			(effects
+				(font
+					(size 1.27 1.27)
+				)
+				(justify left)
+			)
+		)
+		(property "Value" "100nf"
+			(at 275.082 84.836 0)
+			(effects
+				(font
+					(size 1.27 1.27)
+				)
+				(justify left)
+			)
+		)
+		(property "Footprint" ""
+			(at 274.0152 86.36 0)
+			(effects
+				(font
+					(size 1.27 1.27)
+				)
+				(hide yes)
+			)
+		)
+		(property "Datasheet" "~"
+			(at 273.05 82.55 0)
+			(effects
+				(font
+					(size 1.27 1.27)
+				)
+				(hide yes)
+			)
+		)
+		(property "Description" "Unpolarized capacitor"
+			(at 273.05 82.55 0)
+			(effects
+				(font
+					(size 1.27 1.27)
+				)
+				(hide yes)
+			)
+		)
+		(pin "1"
+		)
+		(pin "2"
+		)
+		(instances
+			(project "Devboard-G070-32pins"
+				(path "/64c5f682-8fec-4c85-9390-1583d44cdecc/290b6f7d-8953-4006-b646-06216f45cc7b"
+					(reference "C8")
+					(unit 1)
+				)
+			)
+		)
+	)
+	(symbol
 		(lib_id "Connector_Generic:Conn_02x18_Row_Letter_First")
 		(at 228.6 91.44 0)
@@
 					(unit 1)
 				)
+			)
+		)
+	)
+	(symbol
+		(lib_id "power:GND")
+		(at 273.05 88.9 0)
+		(unit 1)
+		(exclude_from_sim no)
+		(in_bom yes)
+		(on_board yes)
+		(dnp no)
+		(fields_autoplaced yes)
+		(property "Reference" "#PWR06"
+			(at 273.05 95.25 0)
+			(effects
+				(font
+					(size 1.27 1.27)
+				)
+				(hide yes)
+			)
+		)
+		(property "Value" "GND"
+			(at 273.05 93.98 0)
+			(effects
+				(font
+					(size 1.27 1.27)
+				)
+			)
+		)
+		(property "Footprint" ""
+			(at 273.05 88.9 0)
+			(effects
+				(font
+					(size 1.27 1.27)
+				)
+				(hide yes)
+			)
+		)
+		(property "Datasheet" ""
+			(at 273.05 88.9 0)
+			(effects
+				(font
+					(size 1.27 1.27)
+				)
+				(hide yes)
+			)
+		)
+		(property "Description" "Power symbol creates a global label with name \"GND\" , ground"
+			(at 273.05 88.9 0)
+			(effects
+				(font
+					(size 1.27 1.27)
+				)
+				(hide yes)
+			)
+		)
+		(pin "1"
+		)
+		(instances
+			(project "Devboard-G070-32pins"
+				(path "/64c5f682-8fec-4c85-9390-1583d44cdecc/290b6f7d-8953-4006-b646-06216f45cc7b"
+					(reference "#PWR06")
+					(unit 1)
+				)

Commit message: update schematic
Parts:
- J11: footprint (none) -> Connector_PinHeader_2.54mm:PinHeader_1x16_P2.54mm_Vertical
Connections:
- net GND: now also J11.b10 (Pin_b10)
Changed lines of the file:
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@@
 	)
 	(junction
+		(at 85.09 91.44)
+		(diameter 0)
+		(color 0 0 0 0)
+	)
+	(junction
 		(at 110.49 91.44)
 		(diameter 0)
@@
 	(wire
 		(pts
+			(xy 85.09 91.44) (xy 85.09 92.71)
+		)
+		(stroke
+			(width 0)
+			(type default)
+		)
+	)
+	(wire
+		(pts
 			(xy 203.2 96.52) (xy 223.52 96.52)
 		)
@@
 	(wire
 		(pts
-			(xy 85.09 88.9) (xy 85.09 92.71)
+			(xy 85.09 88.9) (xy 85.09 91.44)
 		)
 		(stroke
@@
 	(wire
 		(pts
-			(xy 78.74 91.44) (xy 91.44 91.44)
+			(xy 236.22 96.52) (xy 246.38 96.52)
 		)
 		(stroke
@@
 	(wire
 		(pts
-			(xy 236.22 96.52) (xy 246.38 96.52)
+			(xy 236.22 86.36) (xy 246.38 86.36)
 		)
 		(stroke
@@
 	(wire
 		(pts
-			(xy 236.22 86.36) (xy 246.38 86.36)
+			(xy 104.14 76.2) (xy 120.65 76.2)
 		)
 		(stroke
@@
 	(wire
 		(pts
-			(xy 104.14 76.2) (xy 120.65 76.2)
+			(xy 78.74 106.68) (xy 91.44 106.68)
 		)
 		(stroke
@@
 	(wire
 		(pts
-			(xy 78.74 106.68) (xy 91.44 106.68)
+			(xy 104.14 104.14) (xy 120.65 104.14)
 		)
 		(stroke
@@
 	(wire
 		(pts
-			(xy 104.14 104.14) (xy 120.65 104.14)
+			(xy 85.09 91.44) (xy 91.44 91.44)
 		)
 		(stroke
@@
 			)
 		)
-		(property "Footprint" ""
+		(property "Footprint" "Connector_PinHeader_2.54mm:PinHeader_1x16_P2.54mm_Vertical"
 			(at 99.06 88.9 0)
 			(effects

Commit message: added footprints
Parts:
- C8: footprint (none) -> Capacitor_SMD:C_0201_0603Metric
- J11: footprint Connector_PinHeader_2.54mm:PinHeader_1x16_P2.54mm_Vertical -> Connector_PinHeader_1.00mm:PinHeader_2x08_P1.00mm_Vertical
- J5, J6: footprint (none) -> Connector_PinHeader_1.00mm:PinHeader_1x06_P1.00mm_Vertical
- J7: footprint (none) -> Connector_PinHeader_1.00mm:PinHeader_1x10_P1.00mm_Vertical
- J8: footprint (none) -> Connector_PinHeader_1.00mm:PinHeader_1x08_P1.00mm_Vertical
- J9: footprint (none) -> Connector_PinHeader_1.00mm:PinHeader_2x18_P1.00mm_Vertical
- R5: footprint (none) -> Resistor_SMD:R_0201_0603Metric
Connections:
- net GND: no longer J11.b10 (Pin_b10)
Other:
- moved on the sheet: C8, J11, J5, J6, J7, J8, J9, R5, U3
