File: code.kicad_sch (KiCad schematic)
At the start: 29 parts, among them IC1 MC3479, J1 Conn_01x04, Q3 2N7002H, SW1 SW_MEC_5G, SW3 SW_MEC_5E

Commit message: schematic update
Parts:
- removed C1: 100nF, symbol Device:C
- removed JP5: 2_Open, TestPoint:TestPoint_2Pads_Pitch5.08mm_Drill1.3mm, symbol Jumper:Jumper_2_Open
- removed SW1: SW_MEC_5G, symbol Switch:SW_MEC_5G
- added JP4: 2_Open, TestPoint:TestPoint_2Pads_Pitch5.08mm_Drill1.3mm, symbol Jumper:Jumper_2_Open
Connections:
- net Buzzer: now also JP4.2 (B); no longer R21.1
- new net: JP4.1 (A), R21.1
Other:
- moved on the sheet: C9, R6, R7, SW3

Commit message: added footprints
Parts:
- BZ1: footprint (none) -> Buzzer_Beeper:Buzzer_12x9.5RM7.6
- C9: footprint (none) -> Capacitor_SMD:C_0201_0603Metric
- D1: footprint (none) -> LED_THT:LED_D5.0mm-4_RGB_Wide_Pins
- J1: footprint (none) -> Connector_PinHeader_2.54mm:PinHeader_1x04_P2.54mm_Vertical
- R1, R10, R11, R12, R13, R2, R20, R21, R3, R6, R7, R9: footprint (none) -> Resistor_SMD:R_0201_0603Metric
- R14: footprint (none) -> VResistor_SMD:R_0201_0603Metric
- SW3: footprint (none) -> Button_Switch_THT:SW_PUSH_6mm_H9.5mm
Other:
- moved on the sheet: D1
Changed lines of the file:
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@@
 	(wire
 		(pts
-			(xy 80.01 80.01) (xy 74.93 80.01)
+			(xy 80.01 80.01) (xy 73.66 80.01)
 		)
 		(stroke
@@
 	(wire
 		(pts
-			(xy 64.77 80.01) (xy 59.69 80.01)
+			(xy 63.5 80.01) (xy 59.69 80.01)
 		)
 		(stroke
@@
 	(wire
 		(pts
-			(xy 64.77 90.17) (xy 59.69 90.17)
+			(xy 63.5 90.17) (xy 59.69 90.17)
 		)
 		(stroke
@@
 	(wire
 		(pts
-			(xy 59.69 85.09) (xy 64.77 85.09)
+			(xy 59.69 85.09) (xy 63.5 85.09)
 		)
 		(stroke
@@
 	(wire
 		(pts
-			(xy 80.01 90.17) (xy 74.93 90.17)
+			(xy 80.01 90.17) (xy 73.66 90.17)
 		)
 		(stroke
@@
 	(wire
 		(pts
-			(xy 80.01 85.09) (xy 74.93 85.09)
+			(xy 80.01 85.09) (xy 73.66 85.09)
 		)
 		(stroke
@@
 			)
 		)
-		(property "Footprint" ""
-			(at 145.288 53.34 90)
+		(property "Footprint" "Resistor_SMD:R_0201_0603Metric"
+			(at 146.05 52.07 90)
 			(effects
 				(font
-					(size 1.27 1.27)
+					(size 0.762 0.762)
 				)
-				(hide yes)
 			)
 		)
@@
 			)
 		)
-		(property "Footprint" ""
-			(at 83.82 86.868 90)
+		(property "Footprint" "Resistor_SMD:R_0201_0603Metric"
+			(at 83.82 87.63 90)
 			(effects
 				(font
-					(size 1.27 1.27)
+					(size 0.762 0.762)
 				)
-				(hide yes)
 			)
 		)
@@
 			)
 		)
-		(property "Footprint" ""
-			(at 197.358 72.39 90)
+		(property "Footprint" "Resistor_SMD:R_0201_0603Metric"
+			(at 198.12 71.12 90)
 			(effects
 				(font
-					(size 1.27 1.27)
+					(size 0.762 0.762)
 				)
-				(hide yes)
 			)
 		)
@@
 			)
 		)
-		(property "Footprint" ""
-			(at 182.88 81.788 90)
+		(property "Footprint" "Resistor_SMD:R_0201_0603Metric"
+			(at 182.88 82.55 90)
 			(effects
 				(font
-					(size 1.27 1.27)
+					(size 0.762 0.762)
 				)
-				(hide yes)
 			)
 		)
@@
 			)
 		)
-		(property "Footprint" ""
-			(at 138.43 129.2352 0)
+		(property "Footprint" "Capacitor_SMD:C_0201_0603Metric"
+			(at 142.24 133.35 90)
 			(effects
 				(font
-					(size 1.27 1.27)
+					(size 0.762 0.762)
 				)
-				(hide yes)
 			)
 		)
@@
 		(on_board yes)
 		(dnp no)
-		(fields_autoplaced yes)
 		(property "Reference" "J1"
-			(at 102.87 110.4899 0)
+			(at 102.87 109.8549 0)
 			(effects
 				(font
@@
 		)
 		(property "Value" "Conn_01x04"
-			(at 102.87 113.0299 0)
+			(at 102.87 112.3949 0)
 			(effects
 				(font
@@
 			)
 		)
-		(property "Footprint" ""
-			(at 100.33 110.49 0)
+		(property "Footprint" "Connector_PinHeader_2.54mm:PinHeader_1x04_P2.54mm_Vertical"
+			(at 88.9 119.38 0)
 			(effects
 				(font
-					(size 1.27 1.27)
+					(size 0.762 0.762)
 				)
-				(hide yes)
+				(justify left)
 			)
 		)
@@
 	(symbol
 		(lib_id "Device:LED_RGB")
-		(at 69.85 85.09 0)
+		(at 68.58 85.09 0)
 		(unit 1)
 		(exclude_from_sim no)
@@
 		(dnp no)
 		(property "Reference" "D1"
-			(at 69.85 75.438 0)
+			(at 68.58 75.438 0)
 			(effects
 				(font
@@
 		)
 		(property "Value" "LED_RGB"
-			(at 69.85 93.98 0)
+			(at 68.58 93.98 0)
 			(effects
 				(font
@@
 			)
 		)
-		(property "Footprint" ""
-			(at 69.85 86.36 0)
+		(property "Footprint" "LED_THT:LED_D5.0mm-4_RGB_Wide_Pins"
+			(at 69.85 73.66 0)
 			(effects
 				(font
-					(size 1.27 1.27)
+					(size 0.762 0.762)
 				)
-				(hide yes)
 			)
 		)
 		(property "Datasheet" "~"
-			(at 69.85 86.36 0)
+			(at 68.58 86.36 0)
 			(effects
 				(font
@@
 		)
 		(property "Description" "RGB LED, 6 pin package"
-			(at 69.85 85.09 0)
+			(at 68.58 85.09 0)
 			(effects
 				(font
@@
 			)
 		)
-		(property "Footprint" ""
-			(at 175.768 113.03 90)
+		(property "Footprint" "Resistor_SMD:R_0201_0603Metric"
+			(at 176.53 113.03 90)
 			(effects
 				(font
-					(size 1.27 1.27)
+					(size 0.762 0.762)
 				)
-				(hide yes)
 			)
 		)
@@
 			)
 		)
-		(property "Footprint" ""
-			(at 83.82 91.948 90)
+		(property "Footprint" "Resistor_SMD:R_0201_0603Metric"
+			(at 83.82 93.98 90)
 			(effects
 				(font
-					(size 1.27 1.27)
+					(size 0.762 0.762)
 				)
-				(hide yes)
 			)
 		)
@@
 		(on_board yes)
 		(dnp no)
-		(fields_autoplaced yes)
 		(property "Reference" "SW3"
-			(at 142.24 110.49 0)
+			(at 142.24 109.22 0)
 			(effects
 				(font
@@
 		)
 		(property "Value" "SW_MEC_5E"
-			(at 142.24 113.03 0)
+			(at 142.24 111.76 0)
 			(effects
 				(font
@@
 			)
 		)
-		(property "Footprint" ""
-			(at 142.24 113.03 0)
+		(property "Footprint" "Button_Switch_THT:SW_PUSH_6mm_H9.5mm"
+			(at 142.24 114.3 0)
 			(effects
 				(font
-					(size 1.27 1.27)
+					(size 0.762 0.762)
 				)
-				(hide yes)
 			)
 		)
@@
 			(effects
 				(font
-					(size 1.27 1.27)
+					(size 0.762 0.762)
 					(italic yes)
 				)
 				(justify left)
-				(hide yes)
 			)
 		)
@@
 			)
 		)
-		(property "Footprint" ""
-			(at 81.788 55.88 90)
+		(property "Footprint" "Resistor_SMD:R_0201_0603Metric"
+			(at 80.01 59.69 0)
 			(effects
 				(font
-					(size 1.27 1.27)
+					(size 0.762 0.762)
 				)
-				(hide yes)
 			)
 		)
@@
 			)
 		)
-		(property "Footprint" ""
-			(at 230.378 72.39 90)
+		(property "Footprint" "VResistor_SMD:R_0201_0603Metric"
+			(at 231.14 72.39 90)
 			(effects
 				(font
-					(size 1.27 1.27)
+					(size 0.762 0.762)
 				)
-				(hide yes)
 			)
 		)
@@
 			)
 		)
-		(property "Footprint" ""
+		(property "Footprint" "Resistor_SMD:R_0201_0603Metric"
 			(at 185.42 93.218 90)
 			(effects
 				(font
-					(size 1.27 1.27)
+					(size 0.762 0.762)
 				)
-				(hide yes)
 			)
 		)
@@
 			)
 		)
-		(property "Footprint" ""
-			(at 83.82 81.788 90)
+		(property "Footprint" "Resistor_SMD:R_0201_0603Metric"
+			(at 83.82 82.55 90)
 			(effects
 				(font
-					(size 1.27 1.27)
+					(size 0.762 0.762)
 				)
-				(hide yes)
 			)
 		)
@@
 			)
 		)
-		(property "Footprint" ""
-			(at 138.938 53.34 90)
+		(property "Footprint" "Resistor_SMD:R_0201_0603Metric"
+			(at 132.08 50.8 90)
 			(effects
 				(font
-					(size 1.27 1.27)
+					(size 0.762 0.762)
 				)
-				(hide yes)
 			)
 		)
@@
 			)
 		)
-		(property "Footprint" ""
-			(at 130.048 124.46 90)
+		(property "Footprint" "Resistor_SMD:R_0201_0603Metric"
+			(at 128.27 129.54 0)
 			(effects
 				(font
-					(size 1.27 1.27)
+					(size 0.762 0.762)
 				)
-				(hide yes)
 			)
 		)
@@
 			)
 		)
-		(property "Footprint" ""
-			(at 86.36 49.022 90)
+		(property "Footprint" "Resistor_SMD:R_0201_0603Metric"
+			(at 86.36 46.99 90)
 			(effects
 				(font
-					(size 1.27 1.27)
+					(size 0.762 0.762)
 				)
-				(hide yes)
 			)
 		)
@@
 		)
 		(property "Footprint" "MC3479"
-			(at 247.32 50.8 0)
+			(at 154.94 77.47 90)
 			(effects
 				(font
@@
 				)
 				(justify left top)
-				(hide yes)
 			)
 		)
@@
 			)
 		)
-		(property "Footprint" ""
-			(at 53.975 40.64 90)
+		(property "Footprint" "Buzzer_Beeper:Buzzer_12x9.5RM7.6"
+			(at 53.34 38.1 0)
 			(effects
 				(font
-					(size 1.27 1.27)
+					(size 0.762 0.762)
 				)
-				(hide yes)
 			)
 		)
