File: code.kicad_sch (KiCad schematic)
At the start: 27 parts, among them IC1 MC3479, J1 Conn_01x04, Q3 2N7002H, SW3 SW_MEC_5E

Commit message: [bug] added gnd
Connections:
- net GND: now also C9.2, R6.1
Changed lines of the file:
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@@
+	)
+	(junction
+		(at 132.08 128.27)
+		(diameter 0)
+		(color 0 0 0 0)
 	)
 	(junction
@@
 	(wire
 		(pts
-			(xy 138.43 128.27) (xy 128.27 128.27)
+			(xy 138.43 128.27) (xy 132.08 128.27)
 		)
 		(stroke
@@
 			(width 0)
 			(type dot)
+		)
+	)
+	(wire
+		(pts
+			(xy 132.08 128.27) (xy 128.27 128.27)
+		)
+		(stroke
+			(width 0)
+			(type default)
 		)
 	)
@@
 					(unit 1)
 				)
+			)
+		)
+	)
+	(symbol
+		(lib_id "power:GND")
+		(at 132.08 128.27 0)
+		(unit 1)
+		(exclude_from_sim no)
+		(in_bom yes)
+		(on_board yes)
+		(dnp no)
+		(fields_autoplaced yes)
+		(property "Reference" "#PWR03"
+			(at 132.08 134.62 0)
+			(effects
+				(font
+					(size 1.27 1.27)
+				)
+				(hide yes)
+			)
+		)
+		(property "Value" "GND"
+			(at 132.08 133.35 0)
+			(effects
+				(font
+					(size 1.27 1.27)
+				)
+			)
+		)
+		(property "Footprint" ""
+			(at 132.08 128.27 0)
+			(effects
+				(font
+					(size 1.27 1.27)
+				)
+				(hide yes)
+			)
+		)
+		(property "Datasheet" ""
+			(at 132.08 128.27 0)
+			(effects
+				(font
+					(size 1.27 1.27)
+				)
+				(hide yes)
+			)
+		)
+		(property "Description" "Power symbol creates a global label with name \"GND\" , ground"
+			(at 132.08 128.27 0)
+			(effects
+				(font
+					(size 1.27 1.27)
+				)
+				(hide yes)
+			)
+		)
+		(pin "1"
+		)
+		(instances
+			(project ""
+				(path "/64c5f682-8fec-4c85-9390-1583d44cdecc/92178afa-25e2-4cf5-913d-7d5abb21b57b"
+					(reference "#PWR03")
+					(unit 1)
+				)
