File: micro.kicad_sch (KiCad schematic)
At the start: 11 parts, among them SW4 SW_MEC_5E, Y1 32.768Khz, Y2 8Mhz

Commit message: added footprints
Parts:
- C10, C11, C12, C2, C7: footprint (none) -> Capacitor_SMD:C_0201_0603Metric
- D3: footprint (none) -> LED_SMD:LED_Kingbright_KPBD-3224
- R4, R8: footprint (none) -> Resistor_SMD:R_0201_0603Metric
- SW4: footprint (none) -> Button_Switch_THT:SW_PUSH_6mm_H9.5mm
- Y1, Y2: footprint (none) -> Crystal_SMD_G8-2Pin_3.2x1.5mm
Other:
- moved on the sheet: Y1
Changed lines of the file:
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@@
 	(wire
 		(pts
-			(xy 106.68 119.38) (xy 109.22 119.38)
+			(xy 107.95 119.38) (xy 109.22 119.38)
 		)
 		(stroke
@@
 	(wire
 		(pts
-			(xy 99.06 119.38) (xy 96.52 119.38)
+			(xy 100.33 119.38) (xy 96.52 119.38)
 		)
 		(stroke
@@
 			)
 		)
-		(property "Footprint" ""
+		(property "Footprint" "Resistor_SMD:R_0201_0603Metric"
 			(at 171.45 45.212 90)
 			(effects
 				(font
-					(size 1.27 1.27)
-				)
-				(hide yes)
+					(size 0.762 0.762)
+				)
 			)
 		)
@@
 			)
 		)
-		(property "Footprint" ""
-			(at 140.97 131.7752 0)
-			(effects
-				(font
-					(size 1.27 1.27)
-				)
-				(hide yes)
+		(property "Footprint" "Capacitor_SMD:C_0201_0603Metric"
+			(at 144.526 138.176 90)
+			(effects
+				(font
+					(size 0.762 0.762)
+				)
 			)
 		)
@@
 			)
 		)
-		(property "Footprint" ""
+		(property "Footprint" "Capacitor_SMD:C_0201_0603Metric"
 			(at 192.7352 88.9 0)
 			(effects
 				(font
-					(size 1.27 1.27)
-				)
-				(hide yes)
+					(size 0.762 0.762)
+				)
 			)
 		)
@@
 			)
 		)
-		(property "Footprint" ""
-			(at 154.94 124.46 0)
-			(effects
-				(font
-					(size 1.27 1.27)
-				)
-				(hide yes)
-			)
-		)
-		(property "Datasheet" "~"
+		(property "Footprint" "Crystal_SMD_G8-2Pin_3.2x1.5mm"
+			(at 154.94 120.65 90)
+			(effects
+				(font
+					(size 0.762 0.762)
+				)
+			)
+		)
+		(property "Datasheet" "~https://www.mouser.com/datasheet/2/3/ABS07-3080027.pdf"
 			(at 154.94 124.46 0)
 			(effects
@@
 	(symbol
 		(lib_id "Device:Crystal")
-		(at 102.87 119.38 0)
+		(at 104.14 119.38 0)
 		(mirror x)
 		(unit 1)
@@
 		(dnp no)
 		(property "Reference" "Y1"
-			(at 103.124 123.19 0)
+			(at 104.394 123.19 0)
 			(effects
 				(font
@@
 		)
 		(property "Value" "32.768Khz"
-			(at 103.124 115.57 0)
-			(effects
-				(font
-					(size 1.27 1.27)
-				)
-			)
-		)
-		(property "Footprint" ""
-			(at 102.87 119.38 0)
-			(effects
-				(font
-					(size 1.27 1.27)
-				)
-				(hide yes)
+			(at 104.394 115.57 0)
+			(effects
+				(font
+					(size 1.27 1.27)
+				)
+			)
+		)
+		(property "Footprint" "Crystal_SMD_G8-2Pin_3.2x1.5mm"
+			(at 104.14 123.19 0)
+			(effects
+				(font
+					(size 0.762 0.762)
+				)
 			)
 		)
 		(property "Datasheet" "~"
-			(at 102.87 119.38 0)
+			(at 104.14 119.38 0)
 			(effects
 				(font
@@
 		)
 		(property "Description" "Two pin crystal"
-			(at 102.87 119.38 0)
+			(at 104.14 119.38 0)
 			(effects
 				(font
@@
 			)
 		)
-		(property "Footprint" ""
-			(at 110.1852 129.54 0)
-			(effects
-				(font
-					(size 1.27 1.27)
-				)
-				(hide yes)
+		(property "Footprint" "Capacitor_SMD:C_0201_0603Metric"
+			(at 122.428 125.73 0)
+			(effects
+				(font
+					(size 0.762 0.762)
+				)
 			)
 		)
@@
 		(fields_autoplaced yes)
 		(property "Reference" "R8"
-			(at 167.64 123.1899 0)
+			(at 167.64 122.5549 0)
 			(effects
 				(font
@@
 		)
 		(property "Value" "1M"
-			(at 167.64 125.7299 0)
+			(at 167.64 125.0949 0)
 			(effects
 				(font
@@
 			)
 		)
-		(property "Footprint" ""
-			(at 163.322 124.46 90)
-			(effects
-				(font
-					(size 1.27 1.27)
-				)
-				(hide yes)
+		(property "Footprint" "Resistor_SMD:R_0201_0603Metric"
+			(at 167.64 127 0)
+			(effects
+				(font
+					(size 0.762 0.762)
+				)
+				(justify left)
 			)
 		)
@@
 		(fields_autoplaced yes)
 		(property "Reference" "SW4"
-			(at 179.07 68.58 0)
+			(at 179.07 67.31 0)
 			(effects
 				(font
@@
 		)
 		(property "Value" "SW_MEC_5E"
+			(at 179.07 69.85 0)
+			(effects
+				(font
+					(size 1.27 1.27)
+				)
+			)
+		)
+		(property "Footprint" "Button_Switch_THT:SW_PUSH_6mm_H9.5mm"
 			(at 179.07 71.12 0)
 			(effects
 				(font
-					(size 1.27 1.27)
-				)
-			)
-		)
-		(property "Footprint" ""
-			(at 179.07 71.12 0)
-			(effects
-				(font
-					(size 1.27 1.27)
-				)
-				(hide yes)
+					(size 0.762 0.762)
+				)
 			)
 		)
@@
 			)
 		)
-		(property "Footprint" ""
-			(at 97.4852 129.54 0)
-			(effects
-				(font
-					(size 1.27 1.27)
-				)
-				(hide yes)
+		(property "Footprint" "Capacitor_SMD:C_0201_0603Metric"
+			(at 83.312 125.73 0)
+			(effects
+				(font
+					(size 0.762 0.762)
+				)
 			)
 		)
@@
 			)
 		)
-		(property "Footprint" ""
-			(at 140.97 119.0752 0)
-			(effects
-				(font
-					(size 1.27 1.27)
-				)
-				(hide yes)
+		(property "Footprint" "Capacitor_SMD:C_0201_0603Metric"
+			(at 145.034 110.744 90)
+			(effects
+				(font
+					(size 0.762 0.762)
+				)
 			)
 		)
@@
 		(fields_autoplaced yes)
 		(property "Reference" "D3"
-			(at 190.8175 54.61 0)
+			(at 190.8175 39.37 0)
 			(effects
 				(font
@@
 		)
 		(property "Value" "LED_Red"
-			(at 190.8175 52.07 0)
-			(effects
-				(font
-					(size 1.27 1.27)
-				)
-			)
-		)
-		(property "Footprint" ""
-			(at 189.23 46.99 0)
-			(effects
-				(font
-					(size 1.27 1.27)
-				)
-				(hide yes)
-			)
-		)
+			(at 190.8175 41.91 0)
+			(effects
+				(font
+					(size 1.27 1.27)
+				)
+			)
+		)
+		(property "Footprint" "LED_SMD:LED_Kingbright_KPBD-3224"
+			(at 190.8175 44.45 0)
+			(effects
+				(font
+					(size 0.762 0.762)
+				)
+			)
+		)
