File: power.kicad_sch (KiCad schematic)
At the start: 11 parts, among them J2 USB_C_Receptacle_USB2.0_16P, J4 Conn_01x05, U2 TLV70233_SOT23-5

Commit message: added footprints
Parts:
- removed D5: TVS 5.0, symbol Device:D_Zener_Dual_CommonCathode_KAA_Split
- added D6: TVS 5.0, Diode_SMD:D_0402_1005Metric, symbol Device:D_Zener_Dual_CommonCathode_KAA_Split
- C3: value 100nf -> 100uF; footprint (none) -> Capacitor_SMD:C_0201_0603Metric
- C4, C6: footprint (none) -> Capacitor_SMD:C_0201_0603Metric
- C5: value 100nf -> 10uF; footprint (none) -> Capacitor_SMD:C_0201_0603Metric
- D2, D4: footprint (none) -> Diode_SMD:D_0402_1005Metric
- F1: footprint (none) -> Fuse:Fuse_Bourns_MF-RHT100
- J2: footprint (none) -> Connector_USB:USB_C_Receptacle_GCT_USB4110
- J4: footprint (none) -> Connector_PinHeader_1.00mm:PinHeader_1x05_P1.00mm_Vertical
Connections:
- net GND: now also D6.3 (K)
- net at D4.2 (K), F1.1: now also D6.1 (K)
