File: _autosave-Devboard-G070-32pins.kicad_pcb (KiCad board)
At the start: 2 copper layers, 17 parts, among them J1 Conn_01x05, J2 Conn_01x07, J4 Conn_01x07, J5 Conn_01x02, SW1 SW_MEC_5E, SW3 SW_MEC_5E, U2 STM32G070KBTx

Commit message: [perf] update in footprints
Parts:
- moved BZ1 6.12 mm to (134.7, 139.0)
Changed lines of the file:
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@@
 	(footprint "Buzzer_Beeper:Buzzer_12x9.5RM7.6"
 		(layer "F.Cu")
-		(at 133.5 133)
+		(at 134.7 139)
 		(descr "Generic Buzzer, D12mm height 9.5mm with RM7.6mm")
 		(tags "buzzer")
