File: Devboard-G070-32pins.kicad_sch (KiCad schematic)
At the start: 0 parts

Commit message: add reduced prototype
Other:
- sheet Power  renamed peripherls
- removed sheet Code
- removed sheet Extension connectors
- removed sheet Micro
- added sheet connectors (connectors.kicad_sch)
- sheet peripherls: file power.kicad_sch -> peripherls.kicad_sch
- note added: "- É uma boa pratica não colocar espaço nem acento em nome de qualquer arquivo, assim você fecha brechas para erros. Ex: "Placa projeto com malha GND" -> "ProjetoMalhaGND ou projeto_malha_gnd" - Separe seu projeto em páginas de acordo com suas funçõe ou caracteristicas similares - Se apertar nas páginas abaixo e clicar ena letra E, vera os campos: sheetname e sheetfile. - Sempre colocar os mesmos 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"
- note added: "DICAS"
Changed lines of the file:
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@@
 		(rev "1")
+	)
+	(bus
+		(pts
+			(xy 13.97 34.29) (xy 137.16 34.29)
+		)
+		(stroke
+			(width 0)
+			(type default)
+			(color 255 6 2 1)
+		)
+	)
+	(bus
+		(pts
+			(xy 13.97 17.145) (xy 13.97 34.29)
+		)
+		(stroke
+			(width 0)
+			(type default)
+			(color 255 6 2 1)
+		)
+	)
+	(bus
+		(pts
+			(xy 13.97 17.145) (xy 137.16 17.145)
+		)
+		(stroke
+			(width 0)
+			(type default)
+			(color 255 6 2 1)
+		)
+	)
+	(bus
+		(pts
+			(xy 137.16 34.29) (xy 137.16 17.145)
+		)
+		(stroke
+			(width 0)
+			(type default)
+			(color 255 6 2 1)
+		)
 	)
 	(text "https://stm32world.com/wiki/DIY_STM32_Programmer_(ST-Link/V2-1)#Flash_Unprotected_Bootloader\n"
@@
 		)
 	)
+	(text "DICAS"
+		(exclude_from_sim no)
+		(at 17.78 15.875 0)
+		(effects
+			(font
+				(face "KiCad Font")
+				(size 2 2)
+				(thickness 0.4)
+				(bold yes)
+				(color 255 6 2 1)
+			)
+		)
+	)
+	(text "- É uma boa pratica não colocar espaço nem acento em nome de qualquer arquivo, \n  assim você fecha brechas para erros. Ex: \"Placa projeto com malha GND\" -> \"ProjetoMalhaGND ou projeto_malha_gnd\" \n- Separe seu projeto em páginas de acordo com suas funçõe ou caracteristicas similares \n- Se apertar nas páginas abaixo e clicar ena letra E, vera os campos: sheetname e sheetfile.\n- Sempre colocar os mesmos nomes\n- Percebera que na pasta do seu projeto(diretório) havera um aquivos tera um com extenção .kicad_sch\n- Se por acoso alterar o nome da página, lembre de apagar o arquivo antigo no seu diretório"
+		(exclude_from_sim no)
+		(at 14.605 25.4 0)
+		(effects
+			(font
+				(face "KiCad Font")
+				(size 1.27 1.27)
+				(thickness 0.1588)
+			)
+			(justify left)
+		)
+	)
 	(sheet
-		(at 109.22 78.74)
-		(size 38.1 25.4)
+		(at 97.155 76.2)
+		(size 43.18 26.67)
 		(fields_autoplaced yes)
 		(stroke
@@
 			(color 0 0 0 0.0000)
 		)
-		(property "Sheetname" "Micro"
-			(at 109.22 78.0284 0)
+		(property "Sheetname" "connectors"
+			(at 97.155 75.4884 0)
 			(effects
 				(font
@@
 			)
 		)
-		(property "Sheetfile" "micro.kicad_sch"
-			(at 109.22 104.7246 0)
+		(property "Sheetfile" "connectors.kicad_sch"
+			(at 97.155 103.4546 0)
 			(effects
 				(font
@@
 		)
 		(instances
-			(project "Devboard-G070-32pins"
+			(project "prototipoV1"
 				(path "/64c5f682-8fec-4c85-9390-1583d44cdecc"
 					(page "3")
@@
 	)
 	(sheet
-		(at 206.375 79.375)
-		(size 38.735 24.765)
+		(at 148.59 76.2)
+		(size 40.64 26.67)
 		(fields_autoplaced yes)
 		(stroke
@@
 			(color 0 0 0 0.0000)
 		)
-		(property "Sheetname" "Extension connectors"
-			(at 206.375 78.6634 0)
+		(property "Sheetname" "peripherls"
+			(at 148.59 75.4884 0)
 			(effects
 				(font
@@
 			)
 		)
-		(property "Sheetfile" "ExtensionConnectors.kicad_sch"
-			(at 206.375 104.7246 0)
+		(property "Sheetfile" "peripherls.kicad_sch"
+			(at 148.59 103.4546 0)
 			(effects
 				(font
@@
 		)
 		(instances
-			(project "Devboard-G070-32pins"
-				(path "/64c5f682-8fec-4c85-9390-1583d44cdecc"
-					(page "5")
-				)
-			)
-		)
-	)
-	(sheet
-		(at 157.48 78.74)
-		(size 38.1 25.4)
-		(fields_autoplaced yes)
-		(stroke
-			(width 0.1524)
-			(type solid)
-		)
-		(fill
-			(color 0 0 0 0.0000)
-		)
-		(property "Sheetname" "Code"
-			(at 157.48 78.0284 0)
-			(effects
-				(font
-					(size 1.27 1.27)
-				)
-				(justify left bottom)
-			)
-		)
-		(property "Sheetfile" "code.kicad_sch"
-			(at 157.48 104.7246 0)
-			(effects
-				(font
-					(size 1.27 1.27)
-				)
-				(justify left top)
-			)
-		)
-		(instances
-			(project "Devboard-G070-32pins"
-				(path "/64c5f682-8fec-4c85-9390-1583d44cdecc"
-					(page "4")
-				)
-			)
-		)
-	)
-	(sheet
-		(at 58.42 78.74)
-		(size 38.1 25.4)
-		(fields_autoplaced yes)
-		(stroke
-			(width 0.1524)
-			(type solid)
-		)
-		(fill
-			(color 0 0 0 0.0000)
-		)
-		(property "Sheetname" "Power "
-			(at 58.42 78.0284 0)
-			(effects
-				(font
-					(size 1.27 1.27)
-				)
-				(justify left bottom)
-			)
-		)
-		(property "Sheetfile" "power.kicad_sch"
-			(at 58.42 104.7246 0)
-			(effects
-				(font
-					(size 1.27 1.27)
-				)
-				(justify left top)
-			)
-		)
-		(instances
-			(project "Devboard-G070-32pins"
+			(project "prototipoV1"
 				(path "/64c5f682-8fec-4c85-9390-1583d44cdecc"
 					(page "2")

Commit message: done - V1
Parts:
- added H1, H2: fixing hole, MountingHole:MountingHole_3mm_Pad, symbol Mechanical:MountingHole_Pad
Connections:
- no-connect marks 0 -> 2
Changed lines of the file:
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@@
 		(rev "1")
+	)
+	(no_connect
+		(at 224.79 80.01)
+	)
+	(no_connect
+		(at 207.01 80.01)
 	)
 	(bus
@@
 		)
 	)
+	(symbol
+		(lib_id "Mechanical:MountingHole_Pad")
+		(at 207.01 77.47 0)
+		(unit 1)
+		(exclude_from_sim yes)
+		(in_bom no)
+		(on_board yes)
+		(dnp no)
+		(fields_autoplaced yes)
+		(property "Reference" "H1"
+			(at 209.55 74.9299 0)
+			(effects
+				(font
+					(size 1.27 1.27)
+				)
+				(justify left)
+			)
+		)
+		(property "Value" "fixing hole"
+			(at 209.55 77.4699 0)
+			(effects
+				(font
+					(size 1.27 1.27)
+				)
+				(justify left)
+			)
+		)
+		(property "Footprint" "MountingHole:MountingHole_3mm_Pad"
+			(at 207.01 77.47 0)
+			(effects
+				(font
+					(size 1.27 1.27)
+				)
+				(hide yes)
+			)
+		)
+		(property "Datasheet" "~"
+			(at 207.01 77.47 0)
+			(effects
+				(font
+					(size 1.27 1.27)
+				)
+				(hide yes)
+			)
+		)
+		(property "Description" "Mounting Hole with connection"
+			(at 207.01 77.47 0)
+			(effects
+				(font
+					(size 1.27 1.27)
+				)
+				(hide yes)
+			)
+		)
+		(pin "1"
+		)
+		(instances
+			(project "Devboard-G070-32pins"
+				(path "/64c5f682-8fec-4c85-9390-1583d44cdecc"
+					(reference "H1")
+					(unit 1)
+				)
+			)
+		)
+	)
+	(symbol
+		(lib_id "Mechanical:MountingHole_Pad")
+		(at 224.79 77.47 0)
+		(unit 1)
+		(exclude_from_sim yes)
+		(in_bom no)
+		(on_board yes)
+		(dnp no)
+		(fields_autoplaced yes)
+		(property "Reference" "H2"
+			(at 227.33 74.9299 0)
+			(effects
+				(font
+					(size 1.27 1.27)
+				)
+				(justify left)
+			)
+		)
+		(property "Value" "fixing hole"
+			(at 227.33 77.4699 0)
+			(effects
+				(font
+					(size 1.27 1.27)
+				)
+				(justify left)
+			)
+		)
+		(property "Footprint" "MountingHole:MountingHole_3mm_Pad"
+			(at 224.79 77.47 0)
+			(effects
+				(font
+					(size 1.27 1.27)
+				)
+				(hide yes)
+			)
+		)
+		(property "Datasheet" "~"
+			(at 224.79 77.47 0)
+			(effects
+				(font
+					(size 1.27 1.27)
+				)
+				(hide yes)
+			)
+		)
+		(property "Description" "Mounting Hole with connection"
+			(at 224.79 77.47 0)
+			(effects
+				(font
+					(size 1.27 1.27)
+				)
+				(hide yes)
+			)
+		)
+		(pin "1"
+		)
+		(instances
+			(project "Devboard-G070-32pins"
+				(path "/64c5f682-8fec-4c85-9390-1583d44cdecc"
+					(reference "H2")
+					(unit 1)
+				)
+			)
+		)
+	)

Commit message: perf: 45° micro
Parts:
- H1, H2: footprint MountingHole:MountingHole_3mm_Pad -> personalized:V_1mm
Changed lines of the file:
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@@
 			)
 		)
-		(property "Footprint" "MountingHole:MountingHole_3mm_Pad"
+		(property "Footprint" "personalized:V_1mm"
 			(at 207.01 77.47 0)
 			(effects
@@
 			)
 		)
-		(property "Footprint" "MountingHole:MountingHole_3mm_Pad"
+		(property "Footprint" "personalized:V_1mm"
 			(at 224.79 77.47 0)
 			(effects
