File: connectors.kicad_sch (KiCad schematic)
At the start: 4 parts, among them J1 Conn_01x05, J2 Conn_01x07, J4 Conn_01x07, J5 Conn_01x02

Commit message: [feat] PCB routing
Connections:
- net +3V5 is gone; now on net +3V3: J5.1 (Pin_1)
- net PA0 is gone; now on net PA2: J2.10 (Pin_10)
- net +3V3: now also J1.4 (Pin_4); no longer J1.1 (Pin_1)
- net NRST: now also J1.3 (Pin_3); no longer J1.2 (Pin_2)
- net PA1: now also J2.11 (Pin_11); no longer J2.9 (Pin_9)
- net PA10: now also J2.2 (Pin_2); no longer J4.1 (Pin_1)
- net PA2: no longer J2.7 (Pin_7)
- net PA3: now also J2.9 (Pin_9); no longer J2.8 (Pin_8)
- net PA4: now also J2.8 (Pin_8); no longer J2.6 (Pin_6)
- net PA5: now also J2.7 (Pin_7); no longer J2.5 (Pin_5)
- net PA6: now also J2.6 (Pin_6); no longer J2.4 (Pin_4)
- net PA9: now also J4.1 (Pin_1); no longer J4.3 (Pin_3)
- net PB0: now also J2.4 (Pin_4); no longer J2.3 (Pin_3)
- net PB1: now also J2.3 (Pin_3); no longer J2.2 (Pin_2)
- net PB3: now also J4.3 (Pin_3); no longer J4.4 (Pin_4)
- net PB4: now also J4.4 (Pin_4); no longer J4.5 (Pin_5)
- net PB5: now also J4.5 (Pin_5); no longer J4.6 (Pin_6)
- net PB6: now also J4.6 (Pin_6); no longer J4.7 (Pin_7)
- net PB7: now also J4.7 (Pin_7); no longer J4.8 (Pin_8)
- net PB8: now also J4.8 (Pin_8); no longer J4.9 (Pin_9)
- net PB9: now also J4.9 (Pin_9); no longer J4.10 (Pin_10)
- net PC14: now also J4.10 (Pin_10); no longer J4.11 (Pin_11)
- net PC15: now also J4.11 (Pin_11); no longer J2.11 (Pin_11)
- net SWCLK: now also J1.2 (Pin_2); no longer J1.3 (Pin_3)
- net SWDIO: now also J1.1 (Pin_1); no longer J1.4 (Pin_4)
- new net PA7: J2.5 (Pin_5)
Other:
- moved on the sheet: J1

Commit message: Modifying footprint positions
Connections:
- net +3V3: now also J1.1 (Pin_1); no longer J1.4 (Pin_4)
- net NRST: now also J1.4 (Pin_4); no longer J1.3 (Pin_3)
- net SWDIO: now also J1.3 (Pin_3); no longer J1.1 (Pin_1)
- net PA10 renamed PB2
- net PA9 renamed PA11
- net PC6 renamed PA8
Changed lines of the file:
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@@
+		)
+	)
+	(bus
+		(pts
+			(xy 69.215 74.295) (xy 69.215 123.19)
+		)
+		(stroke
+			(width 0)
+			(type default)
 		)
 	)
 	(wire
 		(pts
-			(xy 154.94 104.14) (xy 144.78 104.14)
-		)
-		(stroke
-			(width 0)
-			(type default)
-		)
-	)
-	(bus
-		(pts
-			(xy 69.215 74.295) (xy 69.215 123.19)
+			(xy 154.94 109.22) (xy 154.94 106.68)
 		)
 		(stroke
@@
 	(wire
 		(pts
-			(xy 154.94 109.22) (xy 154.94 106.68)
+			(xy 154.94 96.52) (xy 154.94 93.98)
 		)
 		(stroke
@@
 		)
 	)
+	(wire
+		(pts
+			(xy 144.78 96.52) (xy 154.94 96.52)
+		)
+		(stroke
+			(width 0)
+			(type default)
+		)
+	)
 	(bus
 		(pts
@@
 			(width 0)
 			(type dot)
-		)
-	)
-	(wire
-		(pts
-			(xy 154.94 93.98) (xy 154.94 104.14)
-		)
-		(stroke
-			(width 0)
-			(type default)
 		)
 	)
@@
 		)
 	)
-	(global_label "PC6"
+	(global_label "PA8"
 		(shape input)
 		(at 187.96 115.57 180)
@@
 		)
 		(property "Intersheetrefs" "${INTERSHEET_REFS}"
-			(at 181.2253 115.57 0)
-			(effects
-				(font
-					(size 1.27 1.27)
-				)
-				(justify right)
-				(hide yes)
-			)
-		)
-	)
-	(global_label "PA9"
+			(at 181.4067 115.57 0)
+			(effects
+				(font
+					(size 1.27 1.27)
+				)
+				(justify right)
+				(hide yes)
+			)
+		)
+	)
+	(global_label "SWDIO"
+		(shape input)
+		(at 144.78 101.6 0)
+		(fields_autoplaced yes)
+		(effects
+			(font
+				(size 1.27 1.27)
+			)
+			(justify left)
+		)
+		(property "Intersheetrefs" "${INTERSHEET_REFS}"
+			(at 153.6314 101.6 0)
+			(effects
+				(font
+					(size 1.27 1.27)
+				)
+				(justify left)
+				(hide yes)
+			)
+		)
+	)
+	(global_label "PA15"
+		(shape input)
+		(at 212.09 113.03 0)
+		(fields_autoplaced yes)
+		(effects
+			(font
+				(size 1.27 1.27)
+			)
+			(justify left)
+		)
+		(property "Intersheetrefs" "${INTERSHEET_REFS}"
+			(at 219.8528 113.03 0)
+			(effects
+				(font
+					(size 1.27 1.27)
+				)
+				(justify left)
+				(hide yes)
+			)
+		)
+	)
+	(global_label "NRST"
+		(shape input)
+		(at 144.78 104.14 0)
+		(fields_autoplaced yes)
+		(effects
+			(font
+				(size 1.27 1.27)
+			)
+			(justify left)
+		)
+		(property "Intersheetrefs" "${INTERSHEET_REFS}"
+			(at 152.5428 104.14 0)
+			(effects
+				(font
+					(size 1.27 1.27)
+				)
+				(justify left)
+				(hide yes)
+			)
+		)
+	)
+	(global_label "PA11"
 		(shape input)
 		(at 212.09 115.57 0)
@@
 		)
 		(property "Intersheetrefs" "${INTERSHEET_REFS}"
-			(at 218.6433 115.57 0)
-			(effects
-				(font
-					(size 1.27 1.27)
-				)
-				(justify left)
-				(hide yes)
-			)
-		)
-	)
-	(global_label "SWDIO"
-		(shape input)
-		(at 144.78 96.52 0)
-		(fields_autoplaced yes)
-		(effects
-			(font
-				(size 1.27 1.27)
-			)
-			(justify left)
-		)
-		(property "Intersheetrefs" "${INTERSHEET_REFS}"
-			(at 153.6314 96.52 0)
-			(effects
-				(font
-					(size 1.27 1.27)
-				)
-				(justify left)
-				(hide yes)
-			)
-		)
-	)
-	(global_label "PA15"
-		(shape input)
-		(at 212.09 113.03 0)
-		(fields_autoplaced yes)
-		(effects
-			(font
-				(size 1.27 1.27)
-			)
-			(justify left)
-		)
-		(property "Intersheetrefs" "${INTERSHEET_REFS}"
-			(at 219.8528 113.03 0)
-			(effects
-				(font
-					(size 1.27 1.27)
-				)
-				(justify left)
-				(hide yes)
-			)
-		)
-	)
-	(global_label "NRST"
-		(shape input)
-		(at 144.78 101.6 0)
-		(fields_autoplaced yes)
-		(effects
-			(font
-				(size 1.27 1.27)
-			)
-			(justify left)
-		)
-		(property "Intersheetrefs" "${INTERSHEET_REFS}"
-			(at 152.5428 101.6 0)
-			(effects
-				(font
-					(size 1.27 1.27)
-				)
-				(justify left)
-				(hide yes)
-			)
-		)
-	)
-	(global_label "PA10"
+			(at 219.8528 115.57 0)
+			(effects
+				(font
+					(size 1.27 1.27)
+				)
+				(justify left)
+				(hide yes)
+			)
+		)
+	)
+	(global_label "PA4"
+		(shape input)
+		(at 187.96 97.79 180)
+		(fields_autoplaced yes)
+		(effects
+			(font
+				(size 1.27 1.27)
+			)
+			(justify right)
+		)
+		(property "Intersheetrefs" "${INTERSHEET_REFS}"
+			(at 181.4067 97.79 0)
+			(effects
+				(font
+					(size 1.27 1.27)
+				)
+				(justify right)
+				(hide yes)
+			)
+		)
+	)
+	(global_label "SWCLK"
+		(shape input)
+		(at 144.78 99.06 0)
+		(fields_autoplaced yes)
+		(effects
+			(font
+				(size 1.27 1.27)
+			)
+			(justify left)
+		)
+		(property "Intersheetrefs" "${INTERSHEET_REFS}"
+			(at 153.9942 99.06 0)
+			(effects
+				(font
+					(size 1.27 1.27)
+				)
+				(justify left)
+				(hide yes)
+			)
+		)
+	)
+	(global_label "PC14"
+		(shape input)
+		(at 212.09 92.71 0)
+		(fields_autoplaced yes)
+		(effects
+			(font
+				(size 1.27 1.27)
+			)
+			(justify left)
+		)
+		(property "Intersheetrefs" "${INTERSHEET_REFS}"
+			(at 220.0342 92.71 0)
+			(effects
+				(font
+					(size 1.27 1.27)
+				)
+				(justify left)
+				(hide yes)
+			)
+		)
+	)
+	(global_label "PB2"
 		(shape input)
 		(at 187.96 113.03 180)
@@
 		)
 		(property "Intersheetrefs" "${INTERSHEET_REFS}"
-			(at 180.1972 113.03 0)
-			(effects
-				(font
-					(size 1.27 1.27)
-				)
-				(justify right)
-				(hide yes)
-			)
-		)
-	)
-	(global_label "PA4"
-		(shape input)
-		(at 187.96 97.79 180)
-		(fields_autoplaced yes)
-		(effects
-			(font
-				(size 1.27 1.27)
-			)
-			(justify right)
-		)
-		(property "Intersheetrefs" "${INTERSHEET_REFS}"
-			(at 181.4067 97.79 0)
-			(effects
-				(font
-					(size 1.27 1.27)
-				)
-				(justify right)
-				(hide yes)
-			)
-		)
-	)
-	(global_label "SWCLK"
-		(shape input)
-		(at 144.78 99.06 0)
-		(fields_autoplaced yes)
-		(effects
-			(font
-				(size 1.27 1.27)
-			)
-			(justify left)
-		)
-		(property "Intersheetrefs" "${INTERSHEET_REFS}"
-			(at 153.9942 99.06 0)
-			(effects
-				(font
-					(size 1.27 1.27)
-				)
-				(justify left)
-				(hide yes)
-			)
-		)
-	)
-	(global_label "PC14"
-		(shape input)
-		(at 212.09 92.71 0)
-		(fields_autoplaced yes)
-		(effects
-			(font
-				(size 1.27 1.27)
-			)
-			(justify left)
-		)
-		(property "Intersheetrefs" "${INTERSHEET_REFS}"
-			(at 220.0342 92.71 0)
-			(effects
-				(font
-					(size 1.27 1.27)
-				)
-				(justify left)
-				(hide yes)
-			)
+			(at 181.2253 113.03 0)
+			(effects
+				(font
+					(size 1.27 1.27)
+				)
+				(justify right)
+				(hide yes)
+			)

Commit message: done - V1
Parts:
- removed J5: Conn_01x02, Connector_PinHeader_2.54mm:PinHeader_1x02_P2.54mm_Vertical, symbol Connector_Generic:Conn_01x02
- added J3: Conn_01x01, TestPoint:TestPoint_THTPad_1.0x1.0mm_Drill0.5mm, symbol Connector_Generic:Conn_01x01
- added J5: HW-769, Connector_PinHeader_2.54mm:PinHeader_1x05_P2.54mm_Vertical, symbol Connector_Generic:Conn_01x05
- added J7: Conn_01x03, Connector_PinHeader_2.54mm:PinHeader_1x03_P2.54mm_Vertical, symbol Connector_Generic:Conn_01x03
Connections:
- net GND: now also J5.5 (Pin_5)
- net PA11 renamed PA12
- net PA12: now also J3.1 (Pin_1)
- new net D+: J5.3 (Pin_3), J7.2 (Pin_2)
- new net D-: J5.2 (Pin_2), J7.1 (Pin_1)
- new net DI: J5.4 (Pin_4), J7.3 (Pin_3)
- new net VBUS: J5.1 (Pin_1)

Commit message: perf: 45° micro
Parts:
- J3: footprint TestPoint:TestPoint_THTPad_1.0x1.0mm_Drill0.5mm -> TestPoint_THTPad_D2.0mm_Drill1.0mm
Connections:
- net PA1: now also J4.11 (Pin_11); no longer J2.11 (Pin_11)
- net PA12: no longer J4.1 (Pin_1)
- net PA15: now also J4.1 (Pin_1); no longer J4.2 (Pin_2)
- net PB3: now also J4.2 (Pin_2); no longer J4.3 (Pin_3)
- net PB4: now also J4.3 (Pin_3); no longer J4.4 (Pin_4)
- net PB5: now also J4.4 (Pin_4); no longer J4.5 (Pin_5)
- net PB6: now also J4.5 (Pin_5); no longer J4.6 (Pin_6)
- net PB7: now also J4.6 (Pin_6); no longer J4.7 (Pin_7)
- net PB8: now also J4.7 (Pin_7); no longer J4.8 (Pin_8)
- net PB9: now also J4.8 (Pin_8); no longer J4.9 (Pin_9)
- net PC14: now also J4.9 (Pin_9); no longer J4.10 (Pin_10)
- net PC15: now also J4.10 (Pin_10); no longer J4.11 (Pin_11)
- new net PA9: J2.11 (Pin_11)
Other:
- moved on the sheet: J3

Commit message: board v1
Parts:
- J3: footprint TestPoint_THTPad_D2.0mm_Drill1.0mm -> personalized:hole
Connections:
- net PA12 is gone; now on net PA1: J3.1 (Pin_1)
- net PA2 is gone; now on net PA5: J2.10 (Pin_10)
- net PA3 is gone; now on net PA6: J2.9 (Pin_9)
- net PA4: now also J2.11 (Pin_11); no longer J2.8 (Pin_8)
- net PA5: no longer J2.7 (Pin_7)
- net PA6: no longer J2.6 (Pin_6)
- net PA7: now also J2.8 (Pin_8); no longer J2.5 (Pin_5)
- net PA8: now also J2.4 (Pin_4); no longer J2.1 (Pin_1)
- net PA9: now also J2.3 (Pin_3); no longer J2.11 (Pin_11)
- net PB0: now also J2.7 (Pin_7); no longer J2.4 (Pin_4)
- net PB1: now also J2.6 (Pin_6); no longer J2.3 (Pin_3)
- net PB2: now also J2.5 (Pin_5); no longer J2.2 (Pin_2)
- new net PA10: J2.1 (Pin_1)
- new net PC6: J2.2 (Pin_2)
Other:
- moved on the sheet: J3
