File: peripherls.kicad_sch (KiCad schematic)
At the start: 21 parts, among them J6 NS6312, Q1 2N7002H, Q3 BD237, SW1 SW_MEC_5E, SW3 SW_MEC_5E, U2 STM32G070KBTx

Commit message: fix: RGB LED symbol
Parts:
- D2: symbol Device:LED_ARGB -> Device:LED_KRGB
Connections:
- net at D2.2 (RA): now also R5.1; no longer R3.1
- net at D2.4 (BA): now also R3.1; no longer R5.1
Other:
- moved on the sheet: D2
Changed lines of the file:
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@@
 	)
 	(symbol
-		(lib_id "Device:LED_ARGB")
-		(at 223.52 101.6 0)
+		(lib_id "Device:LED_KRGB")
+		(at 223.52 101.6 180)
 		(unit 1)
 		(exclude_from_sim no)
@@
 		(dnp no)
 		(property "Reference" "D2"
-			(at 223.52 91.948 0)
+			(at 223.52 111.252 0)
 			(effects
 				(font
@@
 		)
 		(property "Value" "LED_RGB"
-			(at 223.52 110.49 0)
+			(at 223.52 92.71 0)
 			(effects
 				(font
@@
 		)
 		(property "Footprint" "personalized:LED_RGB"
-			(at 223.52 102.87 0)
+			(at 223.52 100.33 0)
 			(effects
 				(font
@@
 		)
 		(property "Datasheet" "~"
-			(at 223.52 102.87 0)
+			(at 223.52 100.33 0)
 			(effects
 				(font
@@
 			)
 		)
-		(property "Description" "RGB LED, anode/red/green/blue"
+		(property "Description" "RGB LED, cathode/red/green/blue"
 			(at 223.52 101.6 0)
 			(effects
